Commit message: TCP and WOBJ defined. Error handler NORUNUNIT. server_robot len check. qt_path bugfix. robot xacro.
Former-commit-id: d0aa35b5657be5007c2b661b39237b90cb8dd46c [formerly 12d1ad757f844362c579d9810b4a4e9d5d1ce744]
Former-commit-id: ee0c6adb0dd76a99991bd0924523bb2a3983ca7a

File: proper_workcell/urdf/abb_robot.xacro (robot description, xacro)
@@ -15,5 +15,5 @@
     <parent link="world"/>
     <child link="irbp_a250/base_link"/>
-    <origin xyz="1.755 0.014 0" rpy="0 0 -${pi/2}" />
+    <origin xyz="1.753 0.0147 -0.0031" rpy="0 0 -${pi/2}" />
   </joint>
   <link name="table0">
