Commit message: Added external axis feedback and bug fix.
Former-commit-id: 0cea29006e6e09721e53d345662ec2832e407ba3 [formerly 894cde3b002bc808fc9438962310c0d49e102628]
Former-commit-id: abc9d7122988bd928575d9b56aa2413e8ca85c25

File: proper_workcell/urdf/irbp_a250.xacro (robot description, xacro)
@@ -87,5 +87,5 @@
     <axis xyz="0 0 1" />
   </joint>
-  <joint name="${name}joint2" type="fixed"> <!--"revolute"-->
+  <joint name="${name}joint2" type="revolute"> <!--"revolute"-->
     <parent link="${name}link_1" />
     <child link="${name}link_2" />
@@ -100,5 +100,5 @@
     <axis xyz="0 1 0" />
   </joint>
-  <joint name="${name}joint4" type="fixed"> <!--"continuous"-->
+  <joint name="${name}joint4" type="continuous"> <!--"continuous"-->
     <parent link="${name}link_3" />
     <child link="${name}link_4" />
