Commit message: Added some routines for testing.
Former-commit-id: def40e259523e59baa04cb97628d23ac425fea04 [formerly ee8429f0b991f3b7bfd5d275d0d0be41e6e4894d]
Former-commit-id: 1c41de54bf1bc6e295f158ca157f566c86b60cbf

File: proper_workcell/urdf/proper_workcell.xacro (robot description, xacro)
@@ -3,5 +3,5 @@
   <property name="pi" value="3.141592654" />
   <xacro:property name="workobject_frame">
-    <origin xyz="1.655 -0.087 0.932" rpy="0 0 0" />
+    <origin xyz="1.550 -0.185 0.930" rpy="0 0 0" />
   </xacro:property>
   <xacro:property name="camera_frame">

File: proper_workcell/urdf/wt03_head.xacro (robot description, xacro)
@@ -3,5 +3,5 @@
   <property name="pi" value="3.141592654" />
   <xacro:property name="tcp_frame">
-    <origin xyz="0.216 -0.022 0.474" rpy="${pi} -1.047197555 ${pi}" />
+    <origin xyz="0.2462 -0.0203 0.4320" rpy="${pi} -1.047197555 ${pi}" />
   </xacro:property>
   <!-- Head -->
