Commit message: Some minor modifications.

File: proper_workcell/urdf/workcell.xacro (robot description, xacro)
@@ -9,5 +9,5 @@
   </xacro:property>
   <xacro:property name="camera_frame">
-    <origin xyz="0.0715 0.2219 0.3248" rpy="-1.148206 0.311297 -2.151468" />
+    <origin xyz="0.1085 0.2266 0.3432" rpy="-1.108786 0.296066 -2.162730" />
   </xacro:property>
   <!-- Robot cell -->

Commit message: Moved workobject relative to the table.

File: proper_workcell/urdf/workcell.xacro (robot description, xacro)
@@ -6,8 +6,8 @@
   </xacro:property>
   <xacro:property name="workobject_frame">
-    <origin xyz="1.550 -0.178 0.9308" rpy="0 0 0" />
+    <origin xyz="-0.19128875 0.19347143 0.10301394" rpy="-0.005628050440181059 0.005713681035339754 -1.5507089198045247" />
   </xacro:property>
   <xacro:property name="camera_frame">
-    <origin xyz="0.1085 0.2266 0.3432" rpy="-1.108786 0.296066 -2.162730" />
+    <origin xyz="0.0981 0.2154 0.357" rpy="-1.1426954999537553 0.3065542584105746 -2.172373016740387" />
   </xacro:property>
   <!-- Robot cell -->
@@ -37,7 +37,8 @@
   <link name="workobject" />
   <joint name="workobject" type="fixed">
-    <parent link="base_link" />
+    <parent link="irbp_a250/tool0"/>
     <child link="workobject" />
     <xacro:insert_block name="workobject_frame" />
+    <axis xyz="0 0 1"/>
   </joint>
   <!-- Camera -->

Commit message: Updated TCP and camera configuration.

File: proper_workcell/urdf/workcell.xacro (robot description, xacro)
@@ -3,11 +3,12 @@
   <property name="pi" value="3.141592654" />
   <xacro:property name="tcp_frame">
-    <origin xyz="0.2462 -0.0203 0.4320" rpy="${pi} -1.047197555 ${pi}" />
+    <origin xyz="0.24646 -0.02439 0.433932" rpy="${pi} -1.047197555 ${pi}" />
   </xacro:property>
   <xacro:property name="workobject_frame">
-    <origin xyz="-0.19128875 0.19347143 0.10301394" rpy="-0.005628050440181059 0.005713681035339754 -1.5507089198045247" />
+    <origin xyz="1.550 -0.185 0.930" rpy="0 0 0" />
+    <!--<origin xyz="-0.19128875 0.19347143 0.10301394" rpy="-0.005628050440181059 0.005713681035339754 -1.5507089198045247" />-->
   </xacro:property>
   <xacro:property name="camera_frame">
-    <origin xyz="0.0981 0.2154 0.357" rpy="-1.1426954999537553 0.3065542584105746 -2.172373016740387" />
+    <origin xyz="0.1032 0.2245 0.3464" rpy="-1.091010543013552 0.3125730462781303 -2.197140695867136" />
   </xacro:property>
   <!-- Robot cell -->
@@ -37,8 +38,9 @@
   <link name="workobject" />
   <joint name="workobject" type="fixed">
-    <parent link="irbp_a250/tool0"/>
+    <parent link="base_link" />
+    <!--<parent link="irbp_a250/tool0"/>-->
     <child link="workobject" />
     <xacro:insert_block name="workobject_frame" />
-    <axis xyz="0 0 1"/>
+    <!--<axis xyz="0 0 1"/>-->
   </joint>
   <!-- Camera -->

Commit message: Added tube .jas files

File: proper_workcell/urdf/workcell.xacro (robot description, xacro)
@@ -10,5 +10,5 @@
   </xacro:property>
   <xacro:property name="camera_frame">
-    <origin xyz="0.1032 0.2245 0.3464" rpy="-1.091010543013552 0.3125730462781303 -2.197140695867136" />
+    <origin xyz="0.1124  0.1471  0.36" rpy="-1.0235306080537976 0.2071367767149199 -1.974280886208384" />
   </xacro:property>
   <!-- Robot cell -->

Commit message: Z distance update: Queue size and sorting lists

File: proper_workcell/urdf/workcell.xacro (robot description, xacro)
@@ -10,5 +10,5 @@
   </xacro:property>
   <xacro:property name="camera_frame">
-    <origin xyz="0.1124  0.1471  0.36" rpy="-1.0235306080537976 0.2071367767149199 -1.974280886208384" />
+    <origin xyz="0.2593  0.1265 -0.0073" rpy="-1.531686220600927 -0.013933220259962117 -2.2243073317011355" />
   </xacro:property>
   <!-- Robot cell -->

Commit message: Cache time test

File: proper_workcell/urdf/workcell.xacro (robot description, xacro)
@@ -10,5 +10,5 @@
   </xacro:property>
   <xacro:property name="camera_frame">
-    <origin xyz="0.2593  0.1265 -0.0073" rpy="-1.531686220600927 -0.013933220259962117 -2.2243073317011355" />
+    <origin xyz="0.136  0.1763 0.0791" rpy="-1.5072035390848944 -0.00663141146519974 -2.1508465856006667" />
   </xacro:property>
   <!-- Robot cell -->
